File: MCP9808/MCP9808.sch (KiCad schematic (older format))
At the start: 21 parts, among them J1 Conn_01x06, J2 Conn_01x04, J3 Conn_01x06, J4 Conn_01x04, U1 MCP9808_MSOP

Commit message: MCP9808 .sch and .pcb update
Address Pins Broken Out
Connections:
- net A2: now reaches A2.1 (A), R3.1, U1.5 (A2)
- net A2: now also J3.6 (Pin_6)
- net A1: now reaches A1.1 (A), R4.1, U1.6 (A1)
- net A1: now also J3.5 (Pin_5)
- net A0: now reaches A0.1 (A), R5.1, U1.7 (A0)
- net A0: now also J3.4 (Pin_4)
Other:
- moved on the sheet: C1
Changed lines of the file:
@@
 L Device:C C1
 U 1 1 5E0038E9
-P 5325 1900
-F 0 "C1" H 5440 1945 50  0000 L CNN
-F 1 "10uF" H 5440 1855 50  0000 L CNN
-F 2 "Capacitor_SMD:C_0805_2012Metric" H 5363 1750 50  0001 C CNN
-F 3 "~" H 5325 1900 50  0001 C CNN
-F 4 "C95841" H 5325 1900 50  0001 C CNN "Part"
-	1    5325 1900
+P 5325 1800
+F 0 "C1" H 5440 1845 50  0000 L CNN
+F 1 "10uF" H 5440 1755 50  0000 L CNN
+F 2 "Capacitor_SMD:C_0805_2012Metric" H 5363 1650 50  0001 C CNN
+F 3 "~" H 5325 1800 50  0001 C CNN
+F 4 "C95841" H 5325 1800 50  0001 C CNN "Part"
+	1    5325 1800
 	1    0    0    -1
 $EndComp
@@
 	3550 800  3825 800
 Wire Wire Line
-	5325 1750 5325 800
+	5325 1650 5325 800
 Wire Wire Line
 	4375 1475 4375 800
@@
 	3575 2850 3850 2850
 Wire Wire Line
-	5325 2050 5325 2850
+	5325 1950 5325 2850
 Wire Wire Line
 	4375 2900 4375 2850
@@
 Text GLabel 1725 2900 2    50   Input ~ 0
 SDA
+Text Label 3650 2075 0    50   ~ 0
+A0
+Text Label 3650 2175 0    50   ~ 0
+A1
+Text Label 3650 2275 0    50   ~ 0
+A2
+Text GLabel 1725 2300 2    50   Input ~ 0
+A2
+Text GLabel 1725 2200 2    50   Input ~ 0
+A1
+Text GLabel 1725 2100 2    50   Input ~ 0
+A0
 $EndSCHEMATC
