File: LIS3MDL/LIS3MDL.sch (KiCad schematic (older format))
At the start: 26 parts, among them J1 Conn_01x06, J2 Conn_01x04, J3 Conn_01x06, J4 Conn_01x04, Q1 BSS138DW, Q2 BSS138DW, U1 AP2127K-3.3

Commit message: Schematic.pdf added
Parts:
- gave numbers to parts that had none: 4
Changed lines of the file:
@@
 DRDY
 $Comp
-L SirBoard_Library:LIS3MDL U?
+L SirBoard_Library:LIS3MDL U2
 U 1 1 5E668B4C
 P 5600 3175
-F 0 "U?" H 5775 3825 50  0000 C CNN
+F 0 "U2" H 5775 3825 50  0000 C CNN
 F 1 "LIS3MDL" H 5900 3725 50  0000 C CNN
 F 2 "Package_LGA:LGA-12_2x2mm_P0.5mm" H 5900 3775 50  0001 C CNN
@@
 $EndComp
 $Comp
-L Device:C C?
+L Device:C C5
 U 1 1 5E68F887
 P 6850 3175
-F 0 "C?" H 6965 3220 50  0000 L CNN
+F 0 "C5" H 6965 3220 50  0000 L CNN
 F 1 "100nF" H 6965 3130 50  0000 L CNN
 F 2 "Capacitor_SMD:C_0603_1608Metric" H 6888 3025 50  0001 C CNN
@@
 $EndComp
 $Comp
-L Device:C C?
+L Device:C C3
 U 1 1 5E6912E4
 P 4475 3175
-F 0 "C?" H 4590 3220 50  0000 L CNN
+F 0 "C3" H 4590 3220 50  0000 L CNN
 F 1 "1uF" H 4590 3130 50  0000 L CNN
 F 2 "Capacitor_SMD:C_0603_1608Metric" H 4513 3025 50  0001 C CNN
@@
 	5550 2450 5550 2625
 $Comp
-L Jumper:SolderJumper_2_Open JP?
+L Jumper:SolderJumper_2_Open JP1
 U 1 1 5E6BA06F
 P 5600 2300
-F 0 "JP?" H 5600 2413 50  0000 C CNN
+F 0 "JP1" H 5600 2413 50  0000 C CNN
 F 1 "SolderJumper_2_Open" H 5600 2413 50  0001 C CNN
 F 2 "Jumper:SolderJumper-2_P1.3mm_Open_RoundedPad1.0x1.5mm" H 5600 2300 50  0001 C CNN
