File: MCP4728/MCP4728.kicad_pcb (KiCad board)
At the start: 2 copper layers, 25.4 x 17.8 mm, 22 parts, among them J1 Conn_01x06, J2 Conn_01x04, J3 Conn_01x06, J4 Conn_01x04, U1 MCP4728

Commit message: Soldermask width adjusted
Other:
- rule solder_mask_min_width: 0.1 -> 0.05
Changed lines of the file:
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@@
   )
   (setup
-    (last_trace_width 0.2)
+    (last_trace_width 0.127)
     (user_trace_width 0.2)
     (user_trace_width 0.25)
@@
     (pad_drill 1)
     (pad_to_mask_clearance 0)
-    (solder_mask_min_width 0.1)
+    (solder_mask_min_width 0.05)
     (aux_axis_origin 0 0)
     (visible_elements 7FFFFFFF)
@@
   (segment (start 55.1956 34.4664) (end 57.626 34.4664) (width 0.25) (layer F.Cu) (net 2))
   (segment (start 54.737 34.925) (end 55.1956 34.4664) (width 0.25) (layer F.Cu) (net 2))
+  (segment (start 64.778 36.711) (end 64.516 36.449) (width 0.25) (layer F.Cu) (net 2))
+  (segment (start 64.778 38.141) (end 64.778 36.711) (width 0.25) (layer F.Cu) (net 2))
+  (via (at 64.516 36.449) (size 0.6) (drill 0.3) (layers F.Cu B.Cu) (net 2))
+  (segment (start 68.692 35.687) (end 67.93 36.449) (width 0.25) (layer B.Cu) (net 2))
+  (segment (start 72.8665 38.6395) (end 72.8665 38.6395) (width 0.25) (layer F.Cu) (net 2))
+  (via (at 72.8665 38.6395) (size 0.6) (drill 0.3) (layers F.Cu B.Cu) (net 2))
+  (segment (start 66.2432 36.449) (end 66.2432 37.2364) (width 0.2) (layer B.Cu) (net 2))
+  (segment (start 67.93 36.449) (end 66.2432 36.449) (width 0.25) (layer B.Cu) (net 2))
+  (segment (start 66.2432 36.449) (end 64.516 36.449) (width 0.25) (layer B.Cu) (net 2))
+  (segment (start 67.6463 38.6395) (end 72.8665 38.6395) (width 0.2) (layer B.Cu) (net 2))
+  (segment (start 66.2432 37.2364) (end 67.6463 38.6395) (width 0.2) (layer B.Cu) (net 2))
   (segment (start 72.477999 42.736401) (end 72.477999 40.171001) (width 0.25) (layer F.Cu) (net 3))
   (segment (start 71.628 43.5864) (end 72.477999 42.736401) (width 0.25) (layer F.Cu) (net 3))
@@
   (segment (start 56.2276 35.4664) (end 57.626 35.4664) (width 0.25) (layer F.Cu) (net 3))
   (segment (start 55.626 36.068) (end 56.2276 35.4664) (width 0.25) (layer F.Cu) (net 3))
+  (segment (start 71.867 35.687) (end 70.724 34.544) (width 0.25) (layer B.Cu) (net 3))
+  (segment (start 70.724 34.544) (end 68.199 34.544) (width 0.25) (layer B.Cu) (net 3))
+  (via (at 65.278 35.687) (size 0.6) (drill 0.3) (layers F.Cu B.Cu) (net 3))
+  (segment (start 68.199 34.544) (end 67.056 35.687) (width 0.25) (layer B.Cu) (net 3))
+  (segment (start 67.056 35.687) (end 65.278 35.687) (width 0.25) (layer B.Cu) (net 3))
+  (segment (start 65.278 35.687) (end 65.278 38.141) (width 0.25) (layer F.Cu) (net 3))
+  (segment (start 74.295 38.354) (end 74.295 38.354) (width 0.25) (layer F.Cu) (net 3))
+  (via (at 74.295 38.354) (size 0.6) (drill 0.3) (layers F.Cu B.Cu) (net 3))
+  (segment (start 70.724 34.544) (end 71.0796 34.1884) (width 0.2) (layer B.Cu) (net 3))
+  (segment (start 71.0796 34.1884) (end 74.9554 34.1884) (width 0.2) (layer B.Cu) (net 3))
+  (segment (start 74.9554 34.1884) (end 75.4888 34.7218) (width 0.2) (layer B.Cu) (net 3))
+  (segment (start 75.4888 37.1602) (end 74.295 38.354) (width 0.2) (layer B.Cu) (net 3))
+  (segment (start 75.4888 34.7218) (end 75.4888 37.1602) (width 0.2) (layer B.Cu) (net 3))
   (segment (start 67.945 35.1535) (end 71.4755 35.1535) (width 0.25) (layer F.Cu) (net 4))
   (segment (start 71.7884 35.4664) (end 72.8665 35.4664) (width 0.25) (layer F.Cu) (net 4))
@@
   (segment (start 69.992 36.534592) (end 68.934592 37.592) (width 0.25) (layer B.Cu) (net 12))
   (segment (start 67.945 37.592) (end 67.945 36.7285) (width 0.25) (layer F.Cu) (net 12))
-  (segment (start 64.778 36.711) (end 64.516 36.449) (width 0.25) (layer F.Cu) (net 2))
-  (segment (start 64.778 38.141) (end 64.778 36.711) (width 0.25) (layer F.Cu) (net 2))
-  (via (at 64.516 36.449) (size 0.6) (drill 0.3) (layers F.Cu B.Cu) (net 2))
-  (segment (start 68.692 35.687) (end 67.93 36.449) (width 0.25) (layer B.Cu) (net 2))
-  (segment (start 72.8665 38.6395) (end 72.8665 38.6395) (width 0.25) (layer F.Cu) (net 2))
-  (via (at 72.8665 38.6395) (size 0.6) (drill 0.3) (layers F.Cu B.Cu) (net 2))
-  (segment (start 66.2432 36.449) (end 66.2432 37.2364) (width 0.2) (layer B.Cu) (net 2))
-  (segment (start 67.93 36.449) (end 66.2432 36.449) (width 0.25) (layer B.Cu) (net 2))
-  (segment (start 66.2432 36.449) (end 64.516 36.449) (width 0.25) (layer B.Cu) (net 2))
-  (segment (start 67.6463 38.6395) (end 72.8665 38.6395) (width 0.2) (layer B.Cu) (net 2))
-  (segment (start 66.2432 37.2364) (end 67.6463 38.6395) (width 0.2) (layer B.Cu) (net 2))
   (via (at 70.866 37.719) (size 0.6) (drill 0.3) (layers F.Cu B.Cu) (net 13))
   (segment (start 71.982592 37.719) (end 70.866 37.719) (width 0.25) (layer B.Cu) (net 13))
@@
   (segment (start 73.167 36.534592) (end 71.982592 37.719) (width 0.25) (layer B.Cu) (net 13))
   (segment (start 70.866 37.719) (end 70.866 36.7285) (width 0.25) (layer F.Cu) (net 13))
-  (segment (start 71.867 35.687) (end 70.724 34.544) (width 0.25) (layer B.Cu) (net 3))
-  (segment (start 70.724 34.544) (end 68.199 34.544) (width 0.25) (layer B.Cu) (net 3))
-  (via (at 65.278 35.687) (size 0.6) (drill 0.3) (layers F.Cu B.Cu) (net 3))
-  (segment (start 68.199 34.544) (end 67.056 35.687) (width 0.25) (layer B.Cu) (net 3))
-  (segment (start 67.056 35.687) (end 65.278 35.687) (width 0.25) (layer B.Cu) (net 3))
-  (segment (start 65.278 35.687) (end 65.278 38.141) (width 0.25) (layer F.Cu) (net 3))
-  (segment (start 74.295 38.354) (end 74.295 38.354) (width 0.25) (layer F.Cu) (net 3))
-  (via (at 74.295 38.354) (size 0.6) (drill 0.3) (layers F.Cu B.Cu) (net 3))
-  (segment (start 70.724 34.544) (end 71.0796 34.1884) (width 0.2) (layer B.Cu) (net 3))
-  (segment (start 71.0796 34.1884) (end 74.9554 34.1884) (width 0.2) (layer B.Cu) (net 3))
-  (segment (start 74.9554 34.1884) (end 75.4888 34.7218) (width 0.2) (layer B.Cu) (net 3))
-  (segment (start 75.4888 37.1602) (end 74.295 38.354) (width 0.2) (layer B.Cu) (net 3))
-  (segment (start 75.4888 34.7218) (end 75.4888 37.1602) (width 0.2) (layer B.Cu) (net 3))
   (zone (net 4) (net_name VCC) (layer B.Cu) (hatch none 0.508)
     (connect_pads (clearance 0.15))
