File: 24LCXXX/24LCXXX.kicad_pcb (KiCad board)
At the start: 2 copper layers, 25.4 x 17.8 mm, 19 parts, among them J1 Conn_01x06, J2 Conn_01x04, J3 Conn_01x06, J4 Conn_01x04, U1 24LC512

Commit message: Soldermask width adjusted
Other:
- rule solder_mask_min_width: 0.1 -> 0.05
Changed lines of the file:
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@@
   )
   (setup
-    (last_trace_width 0.25)
+    (last_trace_width 0.127)
     (user_trace_width 0.2)
     (user_trace_width 0.25)
@@
     (pad_drill 1)
     (pad_to_mask_clearance 0)
-    (solder_mask_min_width 0.1)
+    (solder_mask_min_width 0.05)
     (aux_axis_origin 0 0)
     (visible_elements 7FFFFFFF)
