File: BMI160/BMI160.kicad_pcb (KiCad board)
At the start: 2 copper layers, 25.4 x 17.8 mm, 29 parts, among them J1 Conn_01x06, J2 Conn_01x04, J3 Conn_01x06, J4 Conn_01x04, Q1 BSS138DW, Q2 BSS138DW, U1 AP2127K-3.3, U2 BMI160

Commit message: Soldermask width adjusted
Other:
- rule solder_mask_min_width: 0.1 -> 0.05
Changed lines of the file:
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@@
   )
   (setup
-    (last_trace_width 0.2)
+    (last_trace_width 0.127)
     (user_trace_width 0.2)
     (user_trace_width 0.25)
@@
     (pad_drill 1)
     (pad_to_mask_clearance 0)
-    (solder_mask_min_width 0.1)
+    (solder_mask_min_width 0.05)
     (aux_axis_origin 0 0)
     (visible_elements 7FFFFFFF)
@@
   (segment (start 60.4774 33.8836) (end 61.2902 33.8836) (width 0.2) (layer B.Cu) (net 13))
   (segment (start 61.2902 33.8836) (end 62.1458 33.028) (width 0.2) (layer B.Cu) (net 13))
-  (via (at 63.2714 35.2298) (size 0.6) (drill 0.3) (layers F.Cu B.Cu) (net 14))
-  (segment (start 62.0089 34.9798) (end 63.0214 34.9798) (width 0.2) (layer F.Cu) (net 14))
-  (segment (start 63.0214 34.9798) (end 63.2714 35.2298) (width 0.2) (layer F.Cu) (net 14))
-  (via (at 65.3034 33.7566) (size 0.6) (drill 0.3) (layers F.Cu B.Cu) (net 15))
-  (segment (start 64.5339 34.4798) (end 64.5802 34.4798) (width 0.2) (layer F.Cu) (net 15))
-  (segment (start 64.5802 34.4798) (end 65.3034 33.7566) (width 0.2) (layer F.Cu) (net 15))
-  (segment (start 67.5386 29.8958) (end 69.088 28.3464) (width 0.2) (layer B.Cu) (net 15))
-  (segment (start 66.675 29.8958) (end 67.5386 29.8958) (width 0.2) (layer B.Cu) (net 15))
-  (segment (start 65.3034 33.7566) (end 65.3034 31.2674) (width 0.2) (layer B.Cu) (net 15))
-  (segment (start 65.3034 31.2674) (end 66.675 29.8958) (width 0.2) (layer B.Cu) (net 15))
   (via (at 65.7606 41.3766) (size 0.6) (drill 0.3) (layers F.Cu B.Cu) (net 13))
   (segment (start 66.548 43.5864) (end 66.548 42.164) (width 0.2) (layer B.Cu) (net 13))
@@
   (segment (start 60.4266 33.8986) (end 60.467 33.8582) (width 0.2) (layer B.Cu) (net 13))
   (segment (start 60.4266 35.9664) (end 60.4266 33.8986) (width 0.2) (layer B.Cu) (net 13))
+  (via (at 63.2714 35.2298) (size 0.6) (drill 0.3) (layers F.Cu B.Cu) (net 14))
+  (segment (start 62.0089 34.9798) (end 63.0214 34.9798) (width 0.2) (layer F.Cu) (net 14))
+  (segment (start 63.0214 34.9798) (end 63.2714 35.2298) (width 0.2) (layer F.Cu) (net 14))
   (segment (start 64.0588 34.4424) (end 65.6082 34.4424) (width 0.2) (layer B.Cu) (net 14))
   (segment (start 63.2714 35.2298) (end 64.0588 34.4424) (width 0.2) (layer B.Cu) (net 14))
@@
   (segment (start 70.219201 29.196399) (end 70.778001 29.196399) (width 0.2) (layer B.Cu) (net 14))
   (segment (start 69.596 29.8196) (end 70.219201 29.196399) (width 0.2) (layer B.Cu) (net 14))
+  (via (at 65.3034 33.7566) (size 0.6) (drill 0.3) (layers F.Cu B.Cu) (net 15))
+  (segment (start 64.5339 34.4798) (end 64.5802 34.4798) (width 0.2) (layer F.Cu) (net 15))
+  (segment (start 64.5802 34.4798) (end 65.3034 33.7566) (width 0.2) (layer F.Cu) (net 15))
+  (segment (start 67.5386 29.8958) (end 69.088 28.3464) (width 0.2) (layer B.Cu) (net 15))
+  (segment (start 66.675 29.8958) (end 67.5386 29.8958) (width 0.2) (layer B.Cu) (net 15))
+  (segment (start 65.3034 33.7566) (end 65.3034 31.2674) (width 0.2) (layer B.Cu) (net 15))
+  (segment (start 65.3034 31.2674) (end 66.675 29.8958) (width 0.2) (layer B.Cu) (net 15))
   (zone (net 3) (net_name 3V3) (layer B.Cu) (hatch none 0.508)
     (connect_pads (clearance 0.15))
