File: BMX055/BMX055.kicad_pcb (KiCad board)
At the start: 2 copper layers, 25.4 x 17.8 mm, 30 parts, among them J1 Conn_01x06, J2 Conn_01x04, J3 Conn_01x06, J4 Conn_01x04, Q2 BSS138DW, U1 AP2127K-3.3, U2 BMX055

Commit message: BMX055 - .pcb Updated
Other:
- board text added: "Ax My"
- board text added: "Ay Mx"
- board text removed: "Ax By"
- board text removed: "Ay Bx"
Changed lines of the file:
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@@
   )
   (setup
-    (last_trace_width 0.2)
+    (last_trace_width 0.127)
     (user_trace_width 0.2)
     (user_trace_width 0.25)
@@
     (effects (font (size 0.8 0.8) (thickness 0.12)) (justify left mirror))
   )
-  (gr_text "Ay\nBx" (at 63.6778 32.1818) (layer F.SilkS)
+  (gr_text "Ay\nMx" (at 63.6778 32.1818) (layer F.SilkS)
     (effects (font (size 0.8 0.8) (thickness 0.13)))
   )
@@
     (effects (font (size 0.8 0.8) (thickness 0.13)))
   )
-  (gr_text "Ax\nBy" (at 60.1472 32.1564) (layer F.SilkS)
+  (gr_text "Ax\nMy" (at 60.1472 32.1564) (layer F.SilkS)
     (effects (font (size 0.8 0.8) (thickness 0.13)))
   )

Commit message: Soldermask width adjusted
Other:
- rule solder_mask_min_width: 0.1 -> 0.05
Changed lines of the file:
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@@
     (pad_drill 1)
     (pad_to_mask_clearance 0)
-    (solder_mask_min_width 0.1)
+    (solder_mask_min_width 0.05)
     (aux_axis_origin 0 0)
     (visible_elements 7FFFFFFF)
