File: BNO055/BNO055.sch (KiCad schematic (older format))
At the start: 28 parts, among them J1 Conn_01x06, J2 Conn_01x04, J3 Conn_01x06, J4 Conn_01x04, Q2 BSS138DW, U1 AP2127K-3.3, U2 BNO055, Y1 32.768kHz

Commit message: Part Numbers Added
Parts:
- U2: Part (none) -> C93216
Changed lines of the file:
@@
 F 2 "Package_LGA:LGA-28_5.2x3.8mm_P0.5mm" H 5175 2375 50  0001 L CNN
 F 3 "https://ae-bst.resource.bosch.com/media/_tech/media/datasheets/BST_BNO055_DS000_14.pdf" H 4925 3225 50  0001 C CNN
+F 4 "C93216" H 4925 3025 50  0001 C CNN "Part"
 	1    4925 3025
 	1    0    0    -1

Commit message: Schematic and 3D render updates
Multiple boards
Parts:
- Y1: Part (none) -> C390740
Changed lines of the file:
@@
 F 2 "Crystal:Crystal_SMD_EuroQuartz_EQ161-2Pin_3.2x1.5mm" H 5650 2750 50  0001 C CNN
 F 3 "~" H 5650 2750 50  0001 C CNN
+F 4 "C390740" V 5650 2750 50  0001 C CNN "Part"
 	1    5650 2750
 	0    1    1    0
