File: MCP4725/MCP4725.kicad_pcb (KiCad board)
At the start: 2 copper layers, 25.4 x 17.8 mm, 22 parts, among them J1 Conn_01x06, J2 Conn_01x04, J3 Conn_01x06, J4 Conn_01x04, U1 MCP4725

Commit message: Soldermask width adjusted
Other:
- rule solder_mask_min_width: 0.1 -> 0.05
Changed lines of the file:
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@@
   )
   (setup
-    (last_trace_width 0.2)
+    (last_trace_width 0.127)
     (user_trace_width 0.2)
     (user_trace_width 0.25)
@@
     (pad_drill 1)
     (pad_to_mask_clearance 0)
-    (solder_mask_min_width 0.1)
+    (solder_mask_min_width 0.05)
     (aux_axis_origin 0 0)
     (visible_elements 7FFFFFFF)
@@
   (segment (start 67.691 38.608) (end 69.723 38.608) (width 0.4) (layer B.Cu) (net 1))
   (segment (start 62.357 40.005) (end 65.278 40.005) (width 0.4) (layer B.Cu) (net 1))
-  (segment (start 72.8665 38.6395) (end 72.8665 37.4664) (width 0.25) (layer F.Cu) (net 5))
-  (segment (start 69.088 43.5864) (end 69.088 42.418) (width 0.25) (layer F.Cu) (net 5))
-  (segment (start 69.088 42.418) (end 72.8665 38.6395) (width 0.25) (layer F.Cu) (net 5))
-  (segment (start 69.088 42.384319) (end 68.740681 42.037) (width 0.25) (layer B.Cu) (net 5))
-  (segment (start 69.088 43.5864) (end 69.088 42.384319) (width 0.25) (layer B.Cu) (net 5))
-  (segment (start 68.740681 42.037) (end 59.563 42.037) (width 0.25) (layer B.Cu) (net 5))
-  (via (at 54.737 34.925) (size 0.6) (drill 0.3) (layers F.Cu B.Cu) (net 5))
-  (segment (start 59.563 42.037) (end 54.737 37.211) (width 0.25) (layer B.Cu) (net 5))
-  (segment (start 54.737 37.211) (end 54.737 34.925) (width 0.25) (layer B.Cu) (net 5))
-  (segment (start 55.1956 34.4664) (end 57.626 34.4664) (width 0.25) (layer F.Cu) (net 5))
-  (segment (start 54.737 34.925) (end 55.1956 34.4664) (width 0.25) (layer F.Cu) (net 5))
-  (segment (start 72.477999 42.736401) (end 72.477999 40.171001) (width 0.25) (layer F.Cu) (net 7))
-  (segment (start 71.628 43.5864) (end 72.477999 42.736401) (width 0.25) (layer F.Cu) (net 7))
-  (segment (start 72.477999 40.171001) (end 74.295 38.354) (width 0.25) (layer F.Cu) (net 7))
-  (segment (start 74.295 38.354) (end 74.295 36.83) (width 0.25) (layer F.Cu) (net 7))
-  (segment (start 73.9314 36.4664) (end 72.8665 36.4664) (width 0.25) (layer F.Cu) (net 7))
-  (segment (start 74.295 36.83) (end 73.9314 36.4664) (width 0.25) (layer F.Cu) (net 7))
-  (segment (start 71.628 42.384319) (end 70.264681 41.021) (width 0.25) (layer B.Cu) (net 7))
-  (segment (start 71.628 43.5864) (end 71.628 42.384319) (width 0.25) (layer B.Cu) (net 7))
-  (segment (start 70.264681 41.021) (end 59.563 41.021) (width 0.25) (layer B.Cu) (net 7))
-  (via (at 55.626 36.068) (size 0.6) (drill 0.3) (layers F.Cu B.Cu) (net 7))
-  (segment (start 59.563 41.021) (end 55.626 37.084) (width 0.25) (layer B.Cu) (net 7))
-  (segment (start 55.626 37.084) (end 55.626 36.068) (width 0.25) (layer B.Cu) (net 7))
-  (segment (start 56.2276 35.4664) (end 57.626 35.4664) (width 0.25) (layer F.Cu) (net 7))
-  (segment (start 55.626 36.068) (end 56.2276 35.4664) (width 0.25) (layer F.Cu) (net 7))
   (segment (start 71.7884 35.4664) (end 72.8665 35.4664) (width 0.25) (layer F.Cu) (net 2))
   (segment (start 71.4755 35.1535) (end 71.7884 35.4664) (width 0.25) (layer F.Cu) (net 2))
@@
   (segment (start 69.992 35.687) (end 69.992 36.534592) (width 0.25) (layer B.Cu) (net 4))
   (segment (start 69.992 36.534592) (end 69.061592 37.465) (width 0.25) (layer B.Cu) (net 4))
+  (segment (start 72.8665 38.6395) (end 72.8665 37.4664) (width 0.25) (layer F.Cu) (net 5))
+  (segment (start 69.088 43.5864) (end 69.088 42.418) (width 0.25) (layer F.Cu) (net 5))
+  (segment (start 69.088 42.418) (end 72.8665 38.6395) (width 0.25) (layer F.Cu) (net 5))
+  (segment (start 69.088 42.384319) (end 68.740681 42.037) (width 0.25) (layer B.Cu) (net 5))
+  (segment (start 69.088 43.5864) (end 69.088 42.384319) (width 0.25) (layer B.Cu) (net 5))
+  (segment (start 68.740681 42.037) (end 59.563 42.037) (width 0.25) (layer B.Cu) (net 5))
+  (via (at 54.737 34.925) (size 0.6) (drill 0.3) (layers F.Cu B.Cu) (net 5))
+  (segment (start 59.563 42.037) (end 54.737 37.211) (width 0.25) (layer B.Cu) (net 5))
+  (segment (start 54.737 37.211) (end 54.737 34.925) (width 0.25) (layer B.Cu) (net 5))
+  (segment (start 55.1956 34.4664) (end 57.626 34.4664) (width 0.25) (layer F.Cu) (net 5))
+  (segment (start 54.737 34.925) (end 55.1956 34.4664) (width 0.25) (layer F.Cu) (net 5))
   (segment (start 68.692 35.687) (end 67.183 35.687) (width 0.2) (layer B.Cu) (net 5))
   (via (at 68.707 40.259) (size 0.6) (drill 0.3) (layers F.Cu B.Cu) (net 5))
@@
   (segment (start 73.167 36.534592) (end 71.982592 37.719) (width 0.25) (layer B.Cu) (net 6))
   (segment (start 70.866 37.719) (end 70.866 36.7285) (width 0.25) (layer F.Cu) (net 6))
+  (segment (start 72.477999 42.736401) (end 72.477999 40.171001) (width 0.25) (layer F.Cu) (net 7))
+  (segment (start 71.628 43.5864) (end 72.477999 42.736401) (width 0.25) (layer F.Cu) (net 7))
+  (segment (start 72.477999 40.171001) (end 74.295 38.354) (width 0.25) (layer F.Cu) (net 7))
+  (segment (start 74.295 38.354) (end 74.295 36.83) (width 0.25) (layer F.Cu) (net 7))
+  (segment (start 73.9314 36.4664) (end 72.8665 36.4664) (width 0.25) (layer F.Cu) (net 7))
+  (segment (start 74.295 36.83) (end 73.9314 36.4664) (width 0.25) (layer F.Cu) (net 7))
+  (segment (start 71.628 42.384319) (end 70.264681 41.021) (width 0.25) (layer B.Cu) (net 7))
+  (segment (start 71.628 43.5864) (end 71.628 42.384319) (width 0.25) (layer B.Cu) (net 7))
+  (segment (start 70.264681 41.021) (end 59.563 41.021) (width 0.25) (layer B.Cu) (net 7))
+  (via (at 55.626 36.068) (size 0.6) (drill 0.3) (layers F.Cu B.Cu) (net 7))
+  (segment (start 59.563 41.021) (end 55.626 37.084) (width 0.25) (layer B.Cu) (net 7))
+  (segment (start 55.626 37.084) (end 55.626 36.068) (width 0.25) (layer B.Cu) (net 7))
+  (segment (start 56.2276 35.4664) (end 57.626 35.4664) (width 0.25) (layer F.Cu) (net 7))
+  (segment (start 55.626 36.068) (end 56.2276 35.4664) (width 0.25) (layer F.Cu) (net 7))
   (segment (start 71.342226 36.211774) (end 71.342226 36.226774) (width 0.2) (layer B.Cu) (net 7))
   (segment (start 71.867 35.687) (end 71.342226 36.211774) (width 0.2) (layer B.Cu) (net 7))
