File: TCA9548/TCA9548.kicad_pcb (KiCad board)
At the start: 2 copper layers, 40.6 x 22.9 mm, 39 parts, among them J1 JST_SH_1mm, J10 2.54mm, J2 JST_SH_1mm, J3 JST_SH_1mm, J4 JST_SH_1mm, J5 JST_SH_1mm, J6 JST_SH_1mm, J7 JST_SH_1mm, J8 JST_SH_1mm, J9 JST_SH_1mm

Commit message: Soldermask width adjusted
Other:
- rule solder_mask_min_width: 0.1 -> 0.05
Changed lines of the file:
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@@
   )
   (setup
-    (last_trace_width 0.25)
+    (last_trace_width 0.127)
     (user_trace_width 0.127)
     (user_trace_width 0.15)
@@
     (pad_drill 1)
     (pad_to_mask_clearance 0)
-    (solder_mask_min_width 0.1)
+    (solder_mask_min_width 0.05)
     (aux_axis_origin 0 0)
     (visible_elements 7FFFFFFF)
