File: LTR_303/LTR_303.sch (KiCad schematic (older format))
At the start: 21 parts, among them J1 Conn_01x06, J2 Conn_01x04, J3 Conn_01x06, J4 Conn_01x04, Q1 BSS138DW, Q2 BSS138DW, U1 AP2127K-3.3, U2 LTR-303ALS-01

Commit message: Phew...
almost a screw up
Connections:
- net INT1 is gone; now on net SDA_5V: J3.6 (Pin_6)
- net INT_5V: now also J1.4 (Pin_4), J3.4 (Pin_4)
- net SCL_5V: now also J3.5 (Pin_5)
Changed lines of the file:
@@
 Sheet 1 1
 Title "LTR-303ALS Breakout with 5V Level Shift"
-Date "2020-01-29"
-Rev "1"
+Date "2020-03-10"
+Rev "2"
 Comp "SirBoard"
 Comment1 "Automatic rejection for 50Hz/60Hz lighting"
@@
 Comment4 "LTR-303ALS - SirBlue"
 $EndDescr
-Wire Wire Line
-	5400 1700 5400 1900
-Wire Wire Line
-	5400 1900 6050 1900
-Connection ~ 6050 1900
-Wire Wire Line
-	5750 1175 5400 1175
-Wire Wire Line
-	5400 1175 5400 1275
-Wire Wire Line
-	5400 1275 5750 1275
-Wire Wire Line
-	5400 1275 5400 1400
-Connection ~ 5400 1275
-Wire Wire Line
-	6350 1175 6650 1175
-Wire Wire Line
-	6650 1175 6650 1375
-Text GLabel 5100 1175 0    50   Input ~ 0
-5V
-Wire Wire Line
-	5100 1175 5400 1175
-Connection ~ 5400 1175
-Text GLabel 6975 1175 2    50   Input ~ 0
-3V3
-Connection ~ 6650 1175
-$Comp
-L power:GND #PWR0101
-U 1 1 5DB78905
-P 6050 1975
-F 0 "#PWR0101" H 6050 1725 50  0001 C CNN
-F 1 "GND" H 6054 1803 50  0000 C CNN
-F 2 "" H 6050 1975 50  0001 C CNN
-F 3 "" H 6050 1975 50  0001 C CNN
-	1    6050 1975
-	1    0    0    -1
-$EndComp
-Wire Wire Line
-	6050 1975 6050 1900
 Text GLabel 1400 750  0    50   Input ~ 0
 5V
-Wire Wire Line
-	6650 1900 6050 1900
-Wire Wire Line
-	6650 1675 6650 1900
-$Comp
-L Regulator_Linear:AP2127K-3.3 U1
-U 1 1 5DC7F7BD
-P 6050 1275
-F 0 "U1" H 6050 1615 50  0000 C CNN
-F 1 "AP2127K-3.3" H 6050 1525 50  0000 C CNN
-F 2 "Package_TO_SOT_SMD:SOT-23-5" H 6050 1600 50  0001 C CNN
-F 3 "https://www.diodes.com/assets/Datasheets/AP2127.pdf" H 6050 1375 50  0001 C CNN
-F 4 "C156285" H 6050 1275 50  0001 C CNN "Part"
-	1    6050 1275
-	1    0    0    -1
-$EndComp
-Wire Wire Line
-	6050 1575 6050 1900
 $Comp
 L Device:Q_DUAL_NMOS_S1G1D2S2G2D1 Q1
@@
 	1    0    0    -1
 $EndComp
-Text GLabel 1975 4125 2    50   Input ~ 0
-INT1
 Text GLabel 1250 3825 0    50   Input ~ 0
 GND
-Wire Wire Line
-	6650 1175 6975 1175
 $Comp
 L Mechanical:MountingHole H2
@@
 $EndComp
 $Comp
-L Device:C C1
-U 1 1 5E0038E9
-P 5400 1550
-F 0 "C1" H 5515 1595 50  0000 L CNN
-F 1 "10uF" H 5515 1505 50  0000 L CNN
-F 2 "Capacitor_SMD:C_0805_2012Metric" H 5438 1400 50  0001 C CNN
-F 3 "~" H 5400 1550 50  0001 C CNN
-F 4 "C95841" H 5400 1550 50  0001 C CNN "Part"
-	1    5400 1550
-	1    0    0    -1
-$EndComp
-$Comp
 L Device:Q_DUAL_NMOS_S1G1D2S2G2D1 Q2
 U 1 1 5E08E54B
@@
 Connection ~ 1525 750
 $Comp
-L Device:C C4
-U 1 1 5E37B1B0
-P 6650 1525
-F 0 "C4" H 6765 1570 50  0000 L CNN
-F 1 "10uF" H 6765 1480 50  0000 L CNN
-F 2 "Capacitor_SMD:C_0805_2012Metric" H 6688 1375 50  0001 C CNN
-F 3 "~" H 6650 1525 50  0001 C CNN
-F 4 "C95841" H 6650 1525 50  0001 C CNN "Part"
-	1    6650 1525
-	1    0    0    -1
-$EndComp
-$Comp
 L Connector_Generic:Conn_01x06 J1
 U 1 1 5E3A64F0
@@
 	-1   0    0    -1
 $EndComp
-Text GLabel 1250 4025 0    50   Input ~ 0
-SCL_5V
-Text GLabel 1250 4125 0    50   Input ~ 0
-SDA_5V
 $Comp
 L Connector_Generic:Conn_01x04 J2
@@
 	1    0    0    -1
 $EndComp
+$Comp
+L Device:C C4
+U 1 1 5E37B1B0
+P 6650 1525
+F 0 "C4" H 6765 1570 50  0000 L CNN
+F 1 "10uF" H 6765 1480 50  0000 L CNN
+F 2 "Capacitor_SMD:C_0805_2012Metric" H 6688 1375 50  0001 C CNN
+F 3 "~" H 6650 1525 50  0001 C CNN
+F 4 "C95841" H 6650 1525 50  0001 C CNN "Part"
+	1    6650 1525
+	1    0    0    -1
+$EndComp
+$Comp
+L Device:C C1
+U 1 1 5E0038E9
+P 5400 1550
+F 0 "C1" H 5515 1595 50  0000 L CNN
+F 1 "10uF" H 5515 1505 50  0000 L CNN
+F 2 "Capacitor_SMD:C_0805_2012Metric" H 5438 1400 50  0001 C CNN
+F 3 "~" H 5400 1550 50  0001 C CNN
+F 4 "C95841" H 5400 1550 50  0001 C CNN "Part"
+	1    5400 1550
+	1    0    0    -1
+$EndComp
+Wire Wire Line
+	6650 1175 6975 1175
+Wire Wire Line
+	6050 1575 6050 1900
+$Comp
+L Regulator_Linear:AP2127K-3.3 U1
+U 1 1 5DC7F7BD
+P 6050 1275
+F 0 "U1" H 6050 1615 50  0000 C CNN
+F 1 "AP2127K-3.3" H 6050 1525 50  0000 C CNN
+F 2 "Package_TO_SOT_SMD:SOT-23-5" H 6050 1600 50  0001 C CNN
+F 3 "https://www.diodes.com/assets/Datasheets/AP2127.pdf" H 6050 1375 50  0001 C CNN
+F 4 "C156285" H 6050 1275 50  0001 C CNN "Part"
+	1    6050 1275
+	1    0    0    -1
+$EndComp
+Wire Wire Line
+	6650 1675 6650 1900
+Wire Wire Line
+	6650 1900 6050 1900
+Wire Wire Line
+	6050 1975 6050 1900
+$Comp
+L power:GND #PWR0101
+U 1 1 5DB78905
+P 6050 1975
+F 0 "#PWR0101" H 6050 1725 50  0001 C CNN
+F 1 "GND" H 6054 1803 50  0000 C CNN
+F 2 "" H 6050 1975 50  0001 C CNN
+F 3 "" H 6050 1975 50  0001 C CNN
+	1    6050 1975
+	1    0    0    -1
+$EndComp
+Connection ~ 6650 1175
+Text GLabel 6975 1175 2    50   Input ~ 0
+3V3
+Connection ~ 5400 1175
+Wire Wire Line
+	5100 1175 5400 1175
+Text GLabel 5100 1175 0    50   Input ~ 0
+5V
+Wire Wire Line
+	6650 1175 6650 1375
+Wire Wire Line
+	6350 1175 6650 1175
+Connection ~ 5400 1275
+Wire Wire Line
+	5400 1275 5400 1400
+Wire Wire Line
+	5400 1275 5750 1275
+Wire Wire Line
+	5400 1175 5400 1275
+Wire Wire Line
+	5750 1175 5400 1175
+Connection ~ 6050 1900
+Wire Wire Line
+	5400 1900 6050 1900
+Wire Wire Line
+	5400 1700 5400 1900
+Text GLabel 1975 3925 2    50   Input ~ 0
+INT_5V
+Text GLabel 1250 4125 0    50   Input ~ 0
+SDA_5V
+Text GLabel 1250 4025 0    50   Input ~ 0
+SCL_5V
+Text GLabel 1250 3925 0    50   Input ~ 0
+INT_5V
+Text GLabel 1975 4125 2    50   Input ~ 0
+SDA_5V
+Text GLabel 1975 4025 2    50   Input ~ 0
+SCL_5V
 $EndSCHEMATC

Commit message: Schematic Update - LTR-303
Parts:
- U2: Part (none) -> C364577
Changed lines of the file:
@@
 F 2 "OptoDevice:Lite-On_LTR-303ALS-01" H 5400 3550 50  0001 C CNN
 F 3 "http://optoelectronics.liteon.com/upload/download/DS86-2013-0004/LTR-303ALS-01_DS_V1.pdf" H 5100 3450 50  0001 C CNN
+F 4 "C364577" H 5400 3100 50  0001 C CNN "Part"
 	1    5400 3100
 	1    0    0    -1
