File: DS1307Z/DS1307Z.sch (KiCad schematic (older format))
At the start: 15 parts, among them J1 Conn_01x06, J2 Conn_01x04, J4 Conn_01x04, U1 DS1307ZN+, Y1 32.768kHz

Commit message: DS1307 Update
Bypass Caps Added to Crystal
Parts:
- added C2, C3: 12pF, Capacitor_SMD:C_0603_1608Metric, symbol Device:C
- R1, R2: value 4.7k -> 10k; Part C99782 -> C99198
Connections:
- net GND: now also C2.2, C3.2
- net at U1.1 (X1), Y1.1: now also C2.1
- net at U1.2 (X2), Y1.2: now also C3.1
Other:
- moved on the sheet: Y1
Changed lines of the file:
@@
 EESchema Schematic File Version 4
-LIBS:DS1307Z+-cache
+LIBS:DS1307Z-cache
 EELAYER 29 0
 EELAYER END
@@
 Sheet 1 1
 Title "DS1307Z Breakout "
-Date "2020-02-09"
-Rev "2"
+Date "2020-04-13"
+Rev "2.1"
 Comp "SirBoard"
 Comment1 "www.SirBoard.com"
@@
 L power:GND #PWR0106
 U 1 1 5DCCDF08
-P 4075 2825
-F 0 "#PWR0106" H 4075 2575 50  0001 C CNN
-F 1 "GND" H 4079 2653 50  0000 C CNN
-F 2 "" H 4075 2825 50  0001 C CNN
-F 3 "" H 4075 2825 50  0001 C CNN
-	1    4075 2825
+P 4075 3100
+F 0 "#PWR0106" H 4075 2850 50  0001 C CNN
+F 1 "GND" H 4079 2928 50  0000 C CNN
+F 2 "" H 4075 3100 50  0001 C CNN
+F 3 "" H 4075 3100 50  0001 C CNN
+	1    4075 3100
 	1    0    0    -1
 $EndComp
@@
 P 3175 1450
 F 0 "R2" H 3243 1495 50  0000 L CNN
-F 1 "4.7k" H 3243 1405 50  0000 L CNN
+F 1 "10k" H 3243 1405 50  0000 L CNN
 F 2 "Resistor_SMD:R_0603_1608Metric" V 3215 1440 50  0001 C CNN
 F 3 "~" H 3175 1450 50  0001 C CNN
-F 4 "C99782" H 3175 1450 50  0001 C CNN "Part"
+F 4 "C99198" H 3175 1450 50  0001 C CNN "Part"
 	1    3175 1450
 	1    0    0    -1
@@
 	5075 1750 5075 1225
 Wire Wire Line
-	5075 2050 5075 2750
+	5075 2050 5075 3025
 Wire Wire Line
 	2900 2100 3575 2100
@@
 	3175 2200 3575 2200
 Wire Wire Line
-	4075 2700 4075 2750
-Connection ~ 4075 2750
-Wire Wire Line
-	4075 2750 4075 2825
+	4075 2700 4075 3025
+Connection ~ 4075 3025
+Wire Wire Line
+	4075 3025 4075 3100
 Text GLabel 1000 2100 0    50   Input ~ 0
 SQW
@@
 SCL
 Wire Wire Line
-	4075 2750 4875 2750
+	4075 3025 4875 3025
 $Comp
 L Timer_RTC:DS1307ZN+ U1
@@
 	4700 1550 4875 1550
 Wire Wire Line
-	4875 1550 4875 2750
-Connection ~ 4875 2750
-Wire Wire Line
-	4875 2750 5075 2750
+	4875 1550 4875 3025
+Connection ~ 4875 3025
+Wire Wire Line
+	4875 3025 5075 3025
 $Comp
 L Device:Crystal Y1
 U 1 1 5E423129
-P 3275 2575
-F 0 "Y1" V 3230 2706 50  0000 L CNN
-F 1 "32.768kHz" V 3320 2706 50  0000 L CNN
-F 2 "Crystal:Crystal_SMD_EuroQuartz_EQ161-2Pin_3.2x1.5mm_HandSoldering" H 3275 2575 50  0001 C CNN
-F 3 "~" H 3275 2575 50  0001 C CNN
-F 4 "C390740" V 3275 2575 50  0001 C CNN "Part"
-	1    3275 2575
-	0    -1   1    0
-$EndComp
-Wire Wire Line
-	3575 2400 3275 2400
-Wire Wire Line
-	3275 2400 3275 2425
-Wire Wire Line
-	3275 2725 3275 2750
-Wire Wire Line
-	3275 2750 3525 2750
-Wire Wire Line
-	3525 2750 3525 2500
-Wire Wire Line
-	3525 2500 3575 2500
+P 2850 2525
+F 0 "Y1" H 2800 2250 50  0000 L CNN
+F 1 "32.768kHz" H 2650 2350 50  0000 L CNN
+F 2 "Crystal:Crystal_SMD_EuroQuartz_EQ161-2Pin_3.2x1.5mm_HandSoldering" H 2850 2525 50  0001 C CNN
+F 3 "~" H 2850 2525 50  0001 C CNN
+F 4 "C390740" V 2850 2525 50  0001 C CNN "Part"
+	1    2850 2525
+	1    0    0    1
+$EndComp
 $Comp
 L Device:R_US R1
@@
 P 2900 1450
 F 0 "R1" H 2968 1495 50  0000 L CNN
-F 1 "4.7k" H 2968 1405 50  0000 L CNN
+F 1 "10k" H 2968 1405 50  0000 L CNN
 F 2 "Resistor_SMD:R_0603_1608Metric" V 2940 1440 50  0001 C CNN
 F 3 "~" H 2900 1450 50  0001 C CNN
-F 4 "C99782" H 2900 1450 50  0001 C CNN "Part"
+F 4 "C99198" H 2900 1450 50  0001 C CNN "Part"
 	1    2900 1450
 	1    0    0    -1
@@
 Text Label 4075 1550 0    50   ~ 0
 VBAT
+$Comp
+L Device:C C2
+U 1 1 5EA67C74
+P 2650 2800
+F 0 "C2" H 2765 2845 50  0000 L CNN
+F 1 "12pF" H 2765 2755 50  0000 L CNN
+F 2 "Capacitor_SMD:C_0603_1608Metric" H 2688 2650 50  0001 C CNN
+F 3 "~" H 2650 2800 50  0001 C CNN
+F 4 "C126546" H 2650 2800 50  0001 C CNN "Part"
+	1    2650 2800
+	1    0    0    -1
+$EndComp
+$Comp
+L Device:C C3
+U 1 1 5EA68ABB
+P 3050 2800
+F 0 "C3" H 3165 2845 50  0000 L CNN
+F 1 "12pF" H 3165 2755 50  0000 L CNN
+F 2 "Capacitor_SMD:C_0603_1608Metric" H 3088 2650 50  0001 C CNN
+F 3 "~" H 3050 2800 50  0001 C CNN
+F 4 "C126546" H 3050 2800 50  0001 C CNN "Part"
+	1    3050 2800
+	1    0    0    -1
+$EndComp
+Wire Wire Line
+	2650 2400 3575 2400
+Wire Wire Line
+	2650 2400 2650 2525
+Wire Wire Line
+	2650 2525 2700 2525
+Wire Wire Line
+	2650 2525 2650 2650
+Connection ~ 2650 2525
+Wire Wire Line
+	3050 2500 3050 2525
+Wire Wire Line
+	3000 2525 3050 2525
+Connection ~ 3050 2525
+Wire Wire Line
+	3050 2525 3050 2650
+Wire Wire Line
+	3050 2500 3575 2500
+Wire Wire Line
+	2650 2950 2650 3025
+Wire Wire Line
+	2650 3025 3050 3025
+Wire Wire Line
+	3050 3025 3050 2950
+Wire Wire Line
+	3050 3025 4075 3025
+Connection ~ 3050 3025
 $EndSCHEMATC
